File: CanSat_Camera/CanSat_2019_Kamera.kicad_pcb (KiCad board)
At the start: 2 copper layers, 32.3 x 29.2 mm, 32 parts, among them J1 OV5640 24 Pin 0.5 mm, J2 Camera Out 20 Pin 0.5 mm, U1 TLV75528PDBV, U2 TLV75518PDBV

Commit message: updated files for production
Routing:
- net GND: vias 20 -> 27
Changed lines of the file:
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@@
   (general
     (thickness 1.6)
-    (drawings 16)
-    (tracks 261)
+    (drawings 10)
+    (tracks 268)
     (zones 0)
     (modules 32)
@@
     (42 Eco1.User user hide)
     (43 Eco2.User user hide)
-    (44 Edge.Cuts user hide)
+    (44 Edge.Cuts user)
     (45 Margin user hide)
     (46 B.CrtYd user hide)
@@
       (usegerberadvancedattributes false)
       (creategerberjobfile false)
-      (excludeedgelayer true)
+      (excludeedgelayer false)
       (linewidth 0.100000)
       (plotframeref false)
@@
       (outputformat 1)
       (mirror false)
-      (drillshape 1)
+      (drillshape 0)
       (scaleselection 1)
       (outputdirectory ""))
@@
     )
   )
-  (dimension 31.623 (width 0.12) (layer F.SilkS)
-    (gr_text "31.623 mm" (at 152.4635 43.307) (layer F.SilkS)
-      (effects (font (size 1 1) (thickness 0.15)))
-    )
-    (feature1 (pts (xy 168.275 56.007) (xy 168.275 43.990579)))
-    (feature2 (pts (xy 136.652 56.007) (xy 136.652 43.990579)))
-    (crossbar (pts (xy 136.652 44.577) (xy 168.275 44.577)))
-    (arrow1a (pts (xy 168.275 44.577) (xy 167.148496 45.163421)))
-    (arrow1b (pts (xy 168.275 44.577) (xy 167.148496 43.990579)))
-    (arrow2a (pts (xy 136.652 44.577) (xy 137.778504 45.163421)))
-    (arrow2b (pts (xy 136.652 44.577) (xy 137.778504 43.990579)))
-  )
-  (dimension 28.956 (width 0.12) (layer F.SilkS)
-    (gr_text "28.956 mm" (at 152.527 45.847) (layer F.SilkS)
-      (effects (font (size 1 1) (thickness 0.15)))
-    )
-    (feature1 (pts (xy 167.005 54.61) (xy 167.005 46.530579)))
-    (feature2 (pts (xy 138.049 54.61) (xy 138.049 46.530579)))
-    (crossbar (pts (xy 138.049 47.117) (xy 167.005 47.117)))
-    (arrow1a (pts (xy 167.005 47.117) (xy 165.878496 47.703421)))
-    (arrow1b (pts (xy 167.005 47.117) (xy 165.878496 46.530579)))
-    (arrow2a (pts (xy 138.049 47.117) (xy 139.175504 47.703421)))
-    (arrow2b (pts (xy 138.049 47.117) (xy 139.175504 46.530579)))
-  )
-  (dimension 6.224296 (width 0.12) (layer F.SilkS)
-    (gr_text "6.224 mm" (at 164.212274 88.327443 1.169139328) (layer F.SilkS)
-      (effects (font (size 1 1) (thickness 0.15)))
-    )
-    (feature1 (pts (xy 167.132 78.867) (xy 167.309827 87.580505)))
-    (feature2 (pts (xy 160.909 78.994) (xy 161.086827 87.707505)))
-    (crossbar (pts (xy 161.074861 87.121207) (xy 167.297861 86.994207)))
-    (arrow1a (pts (xy 167.297861 86.994207) (xy 166.183557 87.603491)))
-    (arrow1b (pts (xy 167.297861 86.994207) (xy 166.159626 86.430893)))
-    (arrow2a (pts (xy 161.074861 87.121207) (xy 162.213096 87.684521)))
-    (arrow2b (pts (xy 161.074861 87.121207) (xy 162.189165 86.511923)))
-  )
-  (dimension 3.048 (width 0.12) (layer F.SilkS)
-    (gr_text "3.048 mm" (at 164.084 85.979) (layer F.SilkS)
-      (effects (font (size 1 1) (thickness 0.15)))
-    )
-    (feature1 (pts (xy 165.608 78.994) (xy 165.608 85.295421)))
-    (feature2 (pts (xy 162.56 78.994) (xy 162.56 85.295421)))
-    (crossbar (pts (xy 162.56 84.709) (xy 165.608 84.709)))
-    (arrow1a (pts (xy 165.608 84.709) (xy 164.481496 85.295421)))
-    (arrow1b (pts (xy 165.608 84.709) (xy 164.481496 84.122579)))
-    (arrow2a (pts (xy 162.56 84.709) (xy 163.686504 85.295421)))
-    (arrow2b (pts (xy 162.56 84.709) (xy 163.686504 84.122579)))
-  )
-  (dimension 25.908 (width 0.12) (layer F.SilkS)
-    (gr_text "25.908 mm" (at 171.577 68.961 270) (layer F.SilkS)
-      (effects (font (size 1 1) (thickness 0.15)))
-    )
-    (feature1 (pts (xy 168.402 81.915) (xy 170.893421 81.915)))
-    (feature2 (pts (xy 168.402 56.007) (xy 170.893421 56.007)))
-    (crossbar (pts (xy 170.307 56.007) (xy 170.307 81.915)))
-    (arrow1a (pts (xy 170.307 81.915) (xy 169.720579 80.788496)))
-    (arrow1b (pts (xy 170.307 81.915) (xy 170.893421 80.788496)))
-    (arrow2a (pts (xy 170.307 56.007) (xy 169.720579 57.133504)))
-    (arrow2b (pts (xy 170.307 56.007) (xy 170.893421 57.133504)))
-  )
-  (dimension 28.575 (width 0.12) (layer F.SilkS)
-    (gr_text "28.575 mm" (at 174.244 69.0245 90) (layer F.SilkS)
-      (effects (font (size 1 1) (thickness 0.15)))
-    )
-    (feature1 (pts (xy 167.005 54.737) (xy 173.560421 54.737)))
-    (feature2 (pts (xy 167.005 83.312) (xy 173.560421 83.312)))
-    (crossbar (pts (xy 172.974 83.312) (xy 172.974 54.737)))
-    (arrow1a (pts (xy 172.974 54.737) (xy 173.560421 55.863504)))
-    (arrow1b (pts (xy 172.974 54.737) (xy 172.387579 55.863504)))
-    (arrow2a (pts (xy 172.974 83.312) (xy 173.560421 82.185496)))
-    (arrow2b (pts (xy 172.974 83.312) (xy 172.387579 82.185496)))
-  )
   (gr_line (start 168.656 82.042) (end 168.656 55.88) (layer Edge.Cuts) (width 0.05))
   (gr_line (start 167.132 83.566) (end 168.656 82.042) (layer Edge.Cuts) (width 0.05))
@@
   (via (at 156.972 69.85) (size 0.6) (drill 0.3) (layers F.Cu B.Cu) (net 1))
   (via (at 156.21 59.69) (size 0.6) (drill 0.3) (layers F.Cu B.Cu) (net 1))
+  (via (at 146.86788 73.4822) (size 0.6) (drill 0.3) (layers F.Cu B.Cu) (net 1))
+  (via (at 146.94408 67.35572) (size 0.6) (drill 0.3) (layers F.Cu B.Cu) (net 1))
+  (via (at 147.60956 62.992) (size 0.6) (drill 0.3) (layers F.Cu B.Cu) (net 1))
+  (via (at 159.90316 61.4934) (size 0.6) (drill 0.3) (layers F.Cu B.Cu) (net 1))
+  (via (at 161.14268 62.73292) (size 0.6) (drill 0.3) (layers F.Cu B.Cu) (net 1))
+  (via (at 143.7132 75.35164) (size 0.6) (drill 0.3) (layers F.Cu B.Cu) (net 1))
+  (via (at 162.53968 74.36612) (size 0.6) (drill 0.3) (layers F.Cu B.Cu) (net 1))
   (segment (start 142.113 64.135) (end 142.113 66.421) (width 0.5) (layer F.Cu) (net 2))
   (segment (start 142.113 66.421) (end 142.113 67.564) (width 0.5) (layer F.Cu) (net 2))
